File: electrotactile_adapter.brd (EAGLE design)
At the start: 28.6 x 12.8 mm, 18 parts, among them J3 PAD_SMD_L0.5_W1, J4 PAD_SMD_L0.5_W1, J5 PAD_SMD_L0.5_W1, J6 PAD_SMD_L0.5_W1, J7 1X33_MOLEX_FPC_FPC_RIBBON-CAB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, J8 1X33_MOLEX_FPC_FPC_RIBBON-CAB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

Commit message: Update libraries with metadata.
Parts:
- J7, J8: value 1X33_MOLEX_FPC_FPC_RIBBON-CABLE -> 1x33 Molex Connector
Changed lines of the file:
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@@
 </layers>
 <board>
-<fusionsync huburn="a.cGVyc29uYWw6dWUyOTIwMzJm" projecturn="a.cGVyc29uYWw6dWUyOTIwMzJmIzIwMTgwNzA1MTM4OTE2ODgx" f3durn="urn:adsk.wipprod:dm.lineage:pzvnrGiiR2GwniLKW9x1dQ" pcbguid="03aef2c7-31b8-4e5d-9f0d-0065175a7db2" lastpulledtime="" lastsyncedchangeguid="d6e53b4b-bcc8-419e-8275-0ce6e2009477"/>
+<fusionsync huburn="a.cGVyc29uYWw6dWUyOTIwMzJm" projecturn="a.cGVyc29uYWw6dWUyOTIwMzJmIzIwMTgwNzA1MTM4OTE2ODgx" f3durn="urn:adsk.wipprod:dm.lineage:dwfuecGsQY-6mTX8rZNYVg" pcbguid="f673271f-f7dd-4576-97dc-2e51e04b42ed" lastpulledtime="" lastsyncedchangeguid="f859d070-1f05-12f2-c615-715d602d815e"/>
 <plain>
 <wire x1="-14.3" y1="-6.4" x2="14.3" y2="-6.4" width="0" layer="20"/>
@@
 <element name="JP6" library="PiB_connectors" library_urn="urn:adsk.eagle:library:3661805" package="SMT-JUMPER_3_NO_NO-SILK" package3d_urn="urn:adsk.eagle:package:3661846/1" value="JUMPER-SMT_3_NO_NO-SILK" x="0" y="-5.3" rot="MR0"/>
 <element name="JP7" library="PiB_connectors" package="SMT-JUMPER_2_NO_SILK" value="JUMPER_SMD_2-PAD_NO_SILK" x="0" y="0" rot="MR90"/>
-<element name="J7" library="PiB_connectors" package="_MOLEX-5025983393_FPC_PITCH-0.3MM" package3d_urn="urn:adsk.eagle:package:3945547/2" value="1X33_MOLEX_FPC_FPC_RIBBON-CABLE" x="-12" y="0" rot="R270"/>
-<element name="J8" library="PiB_connectors" package="_MOLEX-5025983393_FPC_PITCH-0.3MM" package3d_urn="urn:adsk.eagle:package:3945547/2" value="1X33_MOLEX_FPC_FPC_RIBBON-CABLE" x="12" y="0" rot="R90"/>
+<element name="J7" library="PiB_connectors" package="_MOLEX-5025983393_FPC_PITCH-0.3MM" package3d_urn="urn:adsk.eagle:package:3945547/2" value="1x33 Molex Connector" x="-12" y="0" rot="R270">
+<attribute name="DATASHEET" value="https://www.molex.com/pdm_docs/sd/5025982593_sd.pdf" x="-12" y="0" size="1.778" layer="27" rot="R270" display="off"/>
+<attribute name="DATASHEET_CABLE" value="https://www.molex.com/pdm_docs/sd/150150423_sd.pdf" x="-12" y="0" size="1.778" layer="27" rot="R270" display="off"/>
+<attribute name="DIST" value="Digikey" x="-12" y="0" size="1.778" layer="27" rot="R270" display="off"/>
+<attribute name="DISTLINK" value="https://www.digikey.com/products/en?keywords=WM9775CT-ND" x="-12" y="0" size="1.778" layer="27" rot="R270" display="off"/>
+<attribute name="DISTLINK_CABLE" value="https://www.digikey.com/products/en?keywords=WM9647-ND" x="-12" y="0" size="1.778" layer="27" rot="R270" display="off"/>
+<attribute name="DISTPN" value="WM9775CT-ND" x="-12" y="0" size="1.778" layer="27" rot="R270" display="off"/>
+<attribute name="DISTPN_CABLE" value="WM9647-ND" x="-12" y="0" size="1.778" layer="27" rot="R270" display="off"/>
+<attribute name="DIST_CABLE" value="Digikey" x="-12" y="0" size="1.778" layer="27" rot="R270" display="off"/>
+<attribute name="MFR" value="Molex, LLC" x="-12" y="0" size="1.778" layer="27" rot="R270" display="off"/>
+<attribute name="MFR_CABLE" value="Molex, LLC" x="-12" y="0" size="1.778" layer="27" rot="R270" display="off"/>
+<attribute name="MPN" value="5025983393" x="-12" y="0" size="1.778" layer="27" rot="R270" display="off"/>
+<attribute name="MPN_CABLE" value="0150150233" x="-12" y="0" size="1.778" layer="27" rot="R270" display="off"/>
+<attribute name="VALUE" value="1x33 Molex Connector" x="-12" y="0" size="1.778" layer="27" rot="R270" display="off"/>
+</element>
+<element name="J8" library="PiB_connectors" package="_MOLEX-5025983393_FPC_PITCH-0.3MM" package3d_urn="urn:adsk.eagle:package:3945547/2" value="1x33 Molex Connector" x="12" y="0" rot="R90">
+<attribute name="DATASHEET" value="https://www.molex.com/pdm_docs/sd/5025982593_sd.pdf" x="12" y="0" size="1.778" layer="27" rot="R90" display="off"/>
+<attribute name="DATASHEET_CABLE" value="https://www.molex.com/pdm_docs/sd/150150423_sd.pdf" x="12" y="0" size="1.778" layer="27" rot="R90" display="off"/>
+<attribute name="DIST" value="Digikey" x="12" y="0" size="1.778" layer="27" rot="R90" display="off"/>
+<attribute name="DISTLINK" value="https://www.digikey.com/products/en?keywords=WM9775CT-ND" x="12" y="0" size="1.778" layer="27" rot="R90" display="off"/>
+<attribute name="DISTLINK_CABLE" value="https://www.digikey.com/products/en?keywords=WM9647-ND" x="12" y="0" size="1.778" layer="27" rot="R90" display="off"/>
+<attribute name="DISTPN" value="WM9775CT-ND" x="12" y="0" size="1.778" layer="27" rot="R90" display="off"/>
+<attribute name="DISTPN_CABLE" value="WM9647-ND" x="12" y="0" size="1.778" layer="27" rot="R90" display="off"/>
+<attribute name="DIST_CABLE" value="Digikey" x="12" y="0" size="1.778" layer="27" rot="R90" display="off"/>
+<attribute name="MFR" value="Molex, LLC" x="12" y="0" size="1.778" layer="27" rot="R90" display="off"/>
+<attribute name="MFR_CABLE" value="Molex, LLC" x="12" y="0" size="1.778" layer="27" rot="R90" display="off"/>
+<attribute name="MPN" value="5025983393" x="12" y="0" size="1.778" layer="27" rot="R90" display="off"/>
+<attribute name="MPN_CABLE" value="0150150233" x="12" y="0" size="1.778" layer="27" rot="R90" display="off"/>
+<attribute name="VALUE" value="1x33 Molex Connector" x="12" y="0" size="1.778" layer="27" rot="R90" display="off"/>
+</element>
 <element name="U$1" library="PiB_logo" package="LRG-LOGO" value="" x="0" y="0" rot="MR0"/>
 </elements>
